File: _autosave-STM32H743VIT6 FC.kicad_sch (KiCad schematic)
At the start: 35 parts, among them J2 DX07S016JA3R1500, SW2 SW_Push, U1 STM32H743VITx, U2 USBLC6-2SC6, U3 ICM-42688-P

Commit message: boom boom
Connections:
- net NRST: no longer names the net of C_RESET1.1, U1.14 (NRST)
Changed lines of the file:
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@@
 	)
 	(junction
-		(at 46.99 80.01)
-		(diameter 0)
-		(color 0 0 0 0)
-	)
-	(junction
 		(at 106.68 78.74)
 		(diameter 0)
@@
 	(wire
 		(pts
-			(xy 41.91 80.01) (xy 46.99 80.01)
-		)
-		(stroke
-			(width 0)
-			(type default)
-		)
-	)
-	(wire
-		(pts
 			(xy 74.93 26.67) (xy 85.09 26.67)
 		)
@@
 		)
 	)
-	(global_label "NRST"
-		(shape input)
-		(at 41.91 80.01 180)
-		(fields_autoplaced yes)
-		(effects
-			(font
-				(size 1.27 1.27)
-			)
-			(justify right)
-		)
-		(property "Intersheetrefs" "${INTERSHEET_REFS}"
-			(at -8.255 -15.875 0)
-			(effects
-				(font
-					(size 1.27 1.27)
-				)
-				(hide yes)
-			)
-		)
-	)
 	(global_label "GYRO_MOSI"
 		(shape input)
@@
 				)
 				(justify left)
+				(hide yes)
 			)
 		)
