File: STM32H743VIT6 FC.kicad_pcb (KiCad board)
At the start: 4 copper layers, 37 x 37 mm, 95 parts, among them J1 USB4730-GF-A_REVA, SW2 Y78B22310FP, U1 TPS54302DDCR, U2 USBLC6-2SC6, U3 TPS54302DDCR

Commit message: usb
Parts:
- moved J1 1.44 mm to (182.3, 114.9)
Changed lines of the file:
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@@
 	(footprint "All:GCT_USB4730-GF-A_REVA"
 		(layer "F.Cu")
-		(at 180.9 115.25 90)
+		(at 182.3089 114.9344 90)
 		(property "Reference" "J1"
 			(at 0 0 90)

Commit message: Changed inductor and added net classes.
Parts:
- 9V_L1: footprint Inductor_SMD:L_0603_1608Metric_Pad1.05x0.95mm_HandSolder -> Inductor_SMD:L_Wuerth_MAPI-5030
- MCU_R1: value 10K -> 10k
- moved 9V_L1 19.1 mm to (130.2, 92.2)
Changed lines of the file:
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@@
 			)
 		)
-		(property "Value" "10K"
+		(property "Value" "10k"
 			(at 0 1.43 0)
 			(layer "F.Fab")
@@
 		)
 	)
-	(footprint "Inductor_SMD:L_0603_1608Metric_Pad1.05x0.95mm_HandSolder"
+	(footprint "Inductor_SMD:L_Wuerth_MAPI-5030"
 		(layer "B.Cu")
-		(at 122.2134 109.6264)
-		(descr "Inductor SMD 0603 (1608 Metric), square (rectangular) end terminal, IPC-7351 nominal with elongated pad for handsoldering. (Body size source: http://www.tortai-tech.com/upload/download/2011102023233369053.pdf), generated with kicad-footprint-generator")
-		(tags "inductor handsolder")
+		(at 130.25 92.25)
+		(descr "Inductor, Wuerth, MAPI-5030, 5.4x5.4x3.1mm, (https://www.we-online.com/en/components/products/WE-MAPI?kicad), generated with kicad-footprint-generator gen_inductor.py")
+		(tags "Würth -SMT")
 		(property "Reference" "9V_L1"
-			(at 0 1.43 180)
+			(at 0 3.65 180)
 			(layer "B.SilkS")
 			(effects
@@
 		)
 		(property "Value" "15u"
-			(at 0 -1.43 180)
+			(at 0 -3.65 180)
 			(layer "B.Fab")
 			(effects
@@
 		)
 		(property "LCSC Part" ""
-			(at 0 0 180)
+			(at 0 0 0)
 			(unlocked yes)
 			(layer "B.Fab")
@@
 		(attr smd)
 		(fp_line
-			(start -0.171267 -0.51)
-			(end 0.171267 -0.51)
+			(start -2.81 3.06)
+			(end 2.81 3.06)
 			(stroke
 				(width 0.12)
@@
 		)
 		(fp_line
-			(start -0.171267 0.51)
-			(end 0.171267 0.51)
+			(start 2.81 -3.06)
+			(end -2.81 -3.06)
 			(stroke
 				(width 0.12)
@@
 		)
 		(fp_line
-			(start -1.65 -0.73)
-			(end -1.65 0.73)
+			(start -3.05 -3.05)
+			(end -3.05 3.05)
 			(stroke
 				(width 0.05)
@@
 		)
 		(fp_line
-			(start -1.65 0.73)
-			(end 1.65 0.73)
+			(start -3.05 3.05)
+			(end -0.85 3.05)
 			(stroke
 				(width 0.05)
@@
 		)
 		(fp_line
-			(start 1.65 -0.73)
-			(end -1.65 -0.73)
+			(start -0.85 -3.05)
+			(end -3.05 -3.05)
 			(stroke
 				(width 0.05)
@@
 		)
 		(fp_line
-			(start 1.65 0.73)
-			(end 1.65 -0.73)
+			(start -0.85 -2.95)
+			(end -0.85 -3.05)
 			(stroke
 				(width 0.05)
@@
 		)
 		(fp_line
-			(start -0.8 -0.4)
-			(end -0.8 0.4)
+			(start -0.85 2.95)
+			(end 0.85 2.95)
 			(stroke
-				(width 0.1)
+				(width 0.05)
 				(type solid)
 			)
-			(layer "B.Fab")
+			(layer "B.CrtYd")
 		)
 		(fp_line
-			(start -0.8 0.4)
-			(end 0.8 0.4)
+			(start -0.85 3.05)
+			(end -0.85 2.95)
 			(stroke
-				(width 0.1)
+				(width 0.05)
 				(type solid)
 			)
-			(layer "B.Fab")
+			(layer "B.CrtYd")
 		)
 		(fp_line
-			(start 0.8 -0.4)
-			(end -0.8 -0.4)
+			(start 0.85 -3.05)
+			(end 0.85 -2.95)
 			(stroke
-				(width 0.1)
+				(width 0.05)
 				(type solid)
 			)
-			(layer "B.Fab")
+			(layer "B.CrtYd")
 		)
 		(fp_line
-			(start 0.8 0.4)
-			(end 0.8 -0.4)
+			(start 0.85 -2.95)
+			(end -0.85 -2.95)
+			(stroke
+				(width 0.05)
+				(type solid)
+			)
+			(layer "B.CrtYd")
+		)
+		(fp_line
+			(start 0.85 2.95)
+			(end 0.85 3.05)
+			(stroke
+				(width 0.05)
+				(type solid)
+			)
+			(layer "B.CrtYd")
+		)
+		(fp_line
+			(start 0.85 3.05)
+			(end 3.05 3.05)
+			(stroke
+				(width 0.05)
+				(type solid)
+			)
+			(layer "B.CrtYd")
+		)
+		(fp_line
+			(start 3.05 -3.05)
+			(end 0.85 -3.05)
+			(stroke
+				(width 0.05)
+				(type solid)
+			)
+			(layer "B.CrtYd")
+		)
+		(fp_line
+			(start 3.05 3.05)
+			(end 3.05 -3.05)
+			(stroke
+				(width 0.05)
+				(type solid)
+			)
+			(layer "B.CrtYd")
+		)
+		(fp_rect
+			(start -2.7 2.7)
+			(end 2.7 -2.7)
 			(stroke
 				(width 0.1)
 				(type solid)
 			)
+			(fill no)
 			(layer "B.Fab")
 		)
@@
 			(effects
 				(font
-					(size 0.4 0.4)
-					(thickness 0.06)
+					(size 1 1)
+					(thickness 0.15)
 				)
 				(justify mirror)
@@
 		)
 		(pad "1" smd roundrect
-			(at -0.875 0)
-			(size 1.05 0.95)
+			(at -1.95 0)
+			(size 1.7 5.6)
 			(layers "B.Cu" "B.Mask" "B.Paste")
-			(roundrect_rratio 0.25)
+			(roundrect_rratio 0.147059)
 			(net 16 "Net-(U3-SW)")
 			(pinfunction "1")
@@
 		)
 		(pad "2" smd roundrect
-			(at 0.875 0)
-			(size 1.05 0.95)
+			(at 1.95 0)
+			(size 1.7 5.6)
 			(layers "B.Cu" "B.Mask" "B.Paste")
-			(roundrect_rratio 0.25)
+			(roundrect_rratio 0.147059)
 			(net 17 "9V_REG")
 			(pinfunction "2")
@@
 		)
 		(embedded_fonts no)
-		(model "${KICAD9_3DMODEL_DIR}/Inductor_SMD.3dshapes/L_0603_1608Metric.step"
+		(model "${KIPRJMOD}/lib/7443845030150.stp"
 			(offset
 				(xyz 0 0 0)

Commit message: Added second inductor.
Parts:
- 5V_L1: footprint Inductor_SMD:L_0603_1608Metric_Pad1.05x0.95mm_HandSolder -> Inductor_SMD:L_Wuerth_MAPI-5030
- moved 5V_L1 12.8 mm to (120.0, 92.0)
Changed lines of the file:
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@@
 		)
 	)
-	(footprint "Inductor_SMD:L_0603_1608Metric_Pad1.05x0.95mm_HandSolder"
+	(footprint "Inductor_SMD:L_Wuerth_MAPI-5030"
 		(layer "B.Cu")
-		(at 117.8634 104.6064)
-		(descr "Inductor SMD 0603 (1608 Metric), square (rectangular) end terminal, IPC-7351 nominal with elongated pad for handsoldering. (Body size source: http://www.tortai-tech.com/upload/download/2011102023233369053.pdf), generated with kicad-footprint-generator")
-		(tags "inductor handsolder")
+		(at 120 92)
+		(descr "Inductor, Wuerth, MAPI-5030, 5.4x5.4x3.1mm, (https://www.we-online.com/en/components/products/WE-MAPI?kicad), generated with kicad-footprint-generator gen_inductor.py")
+		(tags "Würth -SMT")
 		(property "Reference" "5V_L1"
-			(at 0 1.43 180)
+			(at 0 3.65 180)
 			(layer "B.SilkS")
 			(effects
@@
 		)
 		(property "Value" "10u"
-			(at 0 -1.43 180)
+			(at 0 -3.65 180)
 			(layer "B.Fab")
 			(effects
@@
 		)
 		(property "LCSC Part" ""
-			(at 0 0 180)
+			(at 0 0 0)
 			(unlocked yes)
 			(layer "B.Fab")
@@
 		(attr smd)
 		(fp_line
-			(start -0.171267 -0.51)
-			(end 0.171267 -0.51)
+			(start -2.81 3.06)
+			(end 2.81 3.06)
 			(stroke
 				(width 0.12)
@@
 		)
 		(fp_line
-			(start -0.171267 0.51)
-			(end 0.171267 0.51)
+			(start 2.81 -3.06)
+			(end -2.81 -3.06)
 			(stroke
 				(width 0.12)
@@
 		)
 		(fp_line
-			(start -1.65 -0.73)
-			(end -1.65 0.73)
-			(stroke
-				(width 0.05)
-				(type solid)
-			)
-			(layer "B.CrtYd")
-		)
-		(fp_line
-			(start -1.65 0.73)
-			(end 1.65 0.73)
-			(stroke
-				(width 0.05)
-				(type solid)
-			)
-			(layer "B.CrtYd")
-		)
-		(fp_line
-			(start 1.65 -0.73)
-			(end -1.65 -0.73)
-			(stroke
-				(width 0.05)
-				(type solid)
-			)
-			(layer "B.CrtYd")
-		)
-		(fp_line
-			(start 1.65 0.73)
-			(end 1.65 -0.73)
-			(stroke
-				(width 0.05)
-				(type solid)
-			)
-			(layer "B.CrtYd")
-		)
-		(fp_line
-			(start -0.8 -0.4)
-			(end -0.8 0.4)
+			(start -3.05 -3.05)
+			(end -3.05 3.05)
+			(stroke
+				(width 0.05)
+				(type solid)
+			)
+			(layer "B.CrtYd")
+		)
+		(fp_line
+			(start -3.05 3.05)
+			(end -0.85 3.05)
+			(stroke
+				(width 0.05)
+				(type solid)
+			)
+			(layer "B.CrtYd")
+		)
+		(fp_line
+			(start -0.85 -3.05)
+			(end -3.05 -3.05)
+			(stroke
+				(width 0.05)
+				(type solid)
+			)
+			(layer "B.CrtYd")
+		)
+		(fp_line
+			(start -0.85 -2.95)
+			(end -0.85 -3.05)
+			(stroke
+				(width 0.05)
+				(type solid)
+			)
+			(layer "B.CrtYd")
+		)
+		(fp_line
+			(start -0.85 2.95)
+			(end 0.85 2.95)
+			(stroke
+				(width 0.05)
+				(type solid)
+			)
+			(layer "B.CrtYd")
+		)
+		(fp_line
+			(start -0.85 3.05)
+			(end -0.85 2.95)
+			(stroke
+				(width 0.05)
+				(type solid)
+			)
+			(layer "B.CrtYd")
+		)
+		(fp_line
+			(start 0.85 -3.05)
+			(end 0.85 -2.95)
+			(stroke
+				(width 0.05)
+				(type solid)
+			)
+			(layer "B.CrtYd")
+		)
+		(fp_line
+			(start 0.85 -2.95)
+			(end -0.85 -2.95)
+			(stroke
+				(width 0.05)
+				(type solid)
+			)
+			(layer "B.CrtYd")
+		)
+		(fp_line
+			(start 0.85 2.95)
+			(end 0.85 3.05)
+			(stroke
+				(width 0.05)
+				(type solid)
+			)
+			(layer "B.CrtYd")
+		)
+		(fp_line
+			(start 0.85 3.05)
+			(end 3.05 3.05)
+			(stroke
+				(width 0.05)
+				(type solid)
+			)
+			(layer "B.CrtYd")
+		)
+		(fp_line
+			(start 3.05 -3.05)
+			(end 0.85 -3.05)
+			(stroke
+				(width 0.05)
+				(type solid)
+			)
+			(layer "B.CrtYd")
+		)
+		(fp_line
+			(start 3.05 3.05)
+			(end 3.05 -3.05)
+			(stroke
+				(width 0.05)
+				(type solid)
+			)
+			(layer "B.CrtYd")
+		)
+		(fp_rect
+			(start -2.7 2.7)
+			(end 2.7 -2.7)
 			(stroke
 				(width 0.1)
 				(type solid)
 			)
-			(layer "B.Fab")
-		)
-		(fp_line
-			(start -0.8 0.4)
-			(end 0.8 0.4)
-			(stroke
-				(width 0.1)
-				(type solid)
-			)
-			(layer "B.Fab")
-		)
-		(fp_line
-			(start 0.8 -0.4)
-			(end -0.8 -0.4)
-			(stroke
-				(width 0.1)
-				(type solid)
-			)
-			(layer "B.Fab")
-		)
-		(fp_line
-			(start 0.8 0.4)
-			(end 0.8 -0.4)
-			(stroke
-				(width 0.1)
-				(type solid)
-			)
+			(fill no)
 			(layer "B.Fab")
 		)
@@
 			(effects
 				(font
-					(size 0.4 0.4)
-					(thickness 0.06)
+					(size 1 1)
+					(thickness 0.15)
 				)
 				(justify mirror)
@@
 		)
 		(pad "1" smd roundrect
-			(at -0.875 0)
-			(size 1.05 0.95)
+			(at -1.95 0)
+			(size 1.7 5.6)
 			(layers "B.Cu" "B.Mask" "B.Paste")
-			(roundrect_rratio 0.25)
+			(roundrect_rratio 0.147059)
 			(net 10 "Net-(U1-SW)")
 			(pinfunction "1")
@@
 		)
 		(pad "2" smd roundrect
-			(at 0.875 0)
-			(size 1.05 0.95)
+			(at 1.95 0)
+			(size 1.7 5.6)
 			(layers "B.Cu" "B.Mask" "B.Paste")
-			(roundrect_rratio 0.25)
+			(roundrect_rratio 0.147059)
 			(net 11 "5V_REG")
 			(pinfunction "2")
@@
 		)
 		(embedded_fonts no)
-		(model "${KICAD9_3DMODEL_DIR}/Inductor_SMD.3dshapes/L_0603_1608Metric.step"
+		(model "${KIPRJMOD}/lib/7443845030100.stp"
 			(offset
 				(xyz 0 0 0)

Commit message: pads
Parts:
- moved VTX_J1 53.9 mm to (171.2, 136.1), turned to 180 degrees
- moved ESC_J1 46.5 mm to (165.8, 104.3)
- moved GPS_J1 43.7 mm to (160.3, 136.1), turned to 180 degrees
- moved ESC_J2 40.1 mm to (165.8, 103.1)
- moved OTHER_J2 32.0 mm to (148.6, 127.8), turned to 90 degrees
- moved CAM_J2 26.4 mm to (162.0, 105.6), turned to 0 degrees
- moved GPS_J2 18.0 mm to (165.8, 134.9), turned to 180 degrees
- moved USB_D1 11.4 mm to (174.1, 122.7)
- moved MCU_D1 3.98 mm to (177.7, 124.5)
- moved MCU_D2 3.98 mm to (177.7, 126.4)
- moved MCU_D3 3.98 mm to (177.7, 128.3)
- moved 9V_D1 2.87 mm to (174.2, 128.3)
- moved 3V3_D1 2.87 mm to (174.2, 124.5)
- moved 5V_D1 2.87 mm to (174.2, 126.4)
- moved VTX_J2 2.61 mm to (165.8, 137.4), turned to 180 degrees
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
Commit message: ...
Parts:
- moved U1 19.4 mm to (127.7, 131.4), turned to 0 degrees
- moved U3 18.1 mm to (140.3, 131.2)
- moved DEBUG_J2 15.6 mm to (142.1, 117.9), turned to -90 degrees
- moved D0 0.80 mm to (173.2, 119.1)
- moved U2 0.80 mm to (173.3, 115.0)
- moved U_STM32 0.43 mm to (162.1, 119.0)
- moved Y_MCU1 0.29 mm to (151.7, 115.0)
Changed lines of the file:
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@@
 	(footprint "Package_TO_SOT_SMD:SOT-23-6"
 		(layer "F.Cu")
-		(at 172.5 115 180)
+		(at 173.295 114.96 180)
 		(descr "SOT, 6 Pin (JEDEC MO-178 Var AB https://www.jedec.org/document_search?search_api_views_fulltext=MO-178), generated with kicad-footprint-generator ipc_gullwing_generator.py")
 		(tags "SOT TO_SOT_SMD")
@@
 	(footprint "All:OSC_CSTNE8M00G520000R0"
 		(layer "F.Cu")
-		(at 151.37 115.01 -90)
+		(at 151.66 114.96 -90)
 		(property "Reference" "Y_MCU1"
 			(at 0.032 -1.7064 90)
@@
 	(footprint "Package_TO_SOT_SMD:SOT-23"
 		(layer "F.Cu")
-		(at 172.425 119.1875 -90)
+		(at 173.22 119.1475 -90)
 		(descr "SOT, 3 Pin (JEDEC TO-236 Var AB https://www.jedec.org/document_search?search_api_views_fulltext=TO-236), generated with kicad-footprint-generator ipc_gullwing_generator.py")
 		(tags "SOT TO_SOT_SMD")
@@
 	(footprint "Package_QFP:LQFP-100_14x14mm_P0.5mm"
 		(layer "F.Cu")
-		(at 161.62 119.01)
+		(at 162.05 119.02)
 		(descr "LQFP, 100 Pin (https://www.nxp.com/docs/en/package-information/SOT407-1.pdf), generated with kicad-footprint-generator ipc_gullwing_generator.py")
 		(tags "LQFP QFP")
@@
 	(footprint "Package_TO_SOT_SMD:SOT-23-6"
 		(layer "B.Cu")
-		(at 145.1432 148.6948)
+		(at 140.2575 131.25)
 		(descr "SOT, 6 Pin (JEDEC MO-178 Var AB https://www.jedec.org/document_search?search_api_views_fulltext=MO-178), generated with kicad-footprint-generator ipc_gullwing_generator.py")
 		(tags "SOT TO_SOT_SMD")
@@
 	(footprint "Package_TO_SOT_SMD:SOT-23-6"
 		(layer "B.Cu")
-		(at 136.0057 148.8948 90)
+		(at 127.65 131.4025)
 		(descr "SOT, 6 Pin (JEDEC MO-178 Var AB https://www.jedec.org/document_search?search_api_views_fulltext=MO-178), generated with kicad-footprint-generator ipc_gullwing_generator.py")
 		(tags "SOT TO_SOT_SMD")
 		(property "Reference" "U1"
-			(at 0 2.4 90)
+			(at 0 2.4 0)
 			(layer "B.SilkS")
 			(effects
@@
 		)
 		(property "Value" "TPS54302DDCR"
-			(at 0 -2.4 90)
+			(at 0 -2.4 0)
 			(layer "B.Fab")
 			(effects
@@
 		)
 		(property "Datasheet" "https://www.ti.com/lit/ds/symlink/tps54302.pdf"
-			(at 0 0 90)
+			(at 0 0 0)
 			(layer "B.Fab")
 			(hide yes)
@@
 		)
 		(property "Description" "3A, 4.5 to 28V Input, EMI Friendly integrated switch synchronous step-down regulator, pulse-skipping, SOT-23-6"
-			(at 0 0 90)
+			(at 0 0 0)
 			(layer "B.Fab")
 			(hide yes)
@@
 		)
 		(property "LCSC Part" ""
-			(at 0 0 270)
+			(at 0 0 180)
 			(unlocked yes)
 			(layer "B.Fab")
@@
 		(fp_line
 			(start 0 -1.56)
-			(end 0.8 -1.56)
+			(end -0.8 -1.56)
 			(stroke
 				(width 0.12)
@@
 		(fp_line
 			(start 0 -1.56)
-			(end -0.8 -1.56)
+			(end 0.8 -1.56)
 			(stroke
 				(width 0.12)
@@
 		(fp_line
 			(start 0 1.56)
-			(end 0.8 1.56)
+			(end -0.8 1.56)
 			(stroke
 				(width 0.12)
@@
 		(fp_line
 			(start 0 1.56)
-			(end -0.8 1.56)
+			(end 0.8 1.56)
 			(stroke
 				(width 0.12)
@@
 		)
 		(fp_line
-			(start 1.05 -1.7)
-			(end -1.05 -1.7)
+			(start -2.05 -1.5)
+			(end -2.05 1.5)
 			(stroke
 				(width 0.05)
@@
 		)
 		(fp_line
-			(start -1.05 -1.7)
-			(end -1.05 -1.5)
+			(start -2.05 1.5)
+			(end -1.05 1.5)
 			(stroke
 				(width 0.05)
@@
 		)
 		(fp_line
-			(start 2.05 -1.5)
-			(end 1.05 -1.5)
+			(start -1.05 -1.7)
+			(end -1.05 -1.5)
 			(stroke
 				(width 0.05)
@@
 		)
 		(fp_line
-			(start 1.05 -1.5)
-			(end 1.05 -1.7)
+			(start -1.05 -1.5)
+			(end -2.05 -1.5)
 			(stroke
 				(width 0.05)
@@
 		)
 		(fp_line
-			(start -1.05 -1.5)
-			(end -2.05 -1.5)
+			(start -1.05 1.5)
+			(end -1.05 1.7)
 			(stroke
 				(width 0.05)
@@
 		)
 		(fp_line
-			(start -2.05 -1.5)
-			(end -2.05 1.5)
+			(start -1.05 1.7)
+			(end 1.05 1.7)
 			(stroke
 				(width 0.05)
@@
 		)
 		(fp_line
-			(start 2.05 1.5)
-			(end 2.05 -1.5)
+			(start 1.05 -1.7)
+			(end -1.05 -1.7)
 			(stroke
 				(width 0.05)
@@
 		)
 		(fp_line
-			(start 1.05 1.5)
-			(end 2.05 1.5)
+			(start 1.05 -1.5)
+			(end 1.05 -1.7)
 			(stroke
 				(width 0.05)
@@
 		)
 		(fp_line
-			(start -1.05 1.5)
-			(end -1.05 1.7)
+			(start 1.05 1.5)
+			(end 2.05 1.5)
 			(stroke
 				(width 0.05)
@@
 		)
 		(fp_line
-			(start -2.05 1.5)
-			(end -1.05 1.5)
+			(start 1.05 1.7)
+			(end 1.05 1.5)
 			(stroke
 				(width 0.05)
@@
 		)
 		(fp_line
-			(start 1.05 1.7)
-			(end 1.05 1.5)
+			(start 2.05 -1.5)
+			(end 1.05 -1.5)
 			(stroke
 				(width 0.05)
@@
 		)
 		(fp_line
-			(start -1.05 1.7)
-			(end 1.05 1.7)
+			(start 2.05 1.5)
+			(end 2.05 -1.5)
 			(stroke
 				(width 0.05)
@@
 		)
 		(fp_text user "${REFERENCE}"
-			(at 0 0 90)
+			(at 0 0 0)
 			(layer "B.Fab")
 			(effects
@@
 		)
 		(pad "1" smd roundrect
-			(at -1.1375 0.95 90)
+			(at -1.1375 0.95)
 			(size 1.325 0.6)
 			(layers "B.Cu" "B.Mask" "B.Paste")
@@
 		)
 		(pad "2" smd roundrect
-			(at -1.1375 0 90)
+			(at -1.1375 0)
 			(size 1.325 0.6)
 			(layers "B.Cu" "B.Mask" "B.Paste")
@@
 		)
 		(pad "3" smd roundrect
-			(at -1.1375 -0.95 90)
+			(at -1.1375 -0.95)
 			(size 1.325 0.6)
 			(layers "B.Cu" "B.Mask" "B.Paste")
@@
 		)
 		(pad "4" smd roundrect
-			(at 1.1375 -0.95 90)
+			(at 1.1375 -0.95)
 			(size 1.325 0.6)
 			(layers "B.Cu" "B.Mask" "B.Paste")
@@
 		)
 		(pad "5" smd roundrect
-			(at 1.1375 0 90)
+			(at 1.1375 0)
 			(size 1.325 0.6)
 			(layers "B.Cu" "B.Mask" "B.Paste")
@@
 		)
 		(pad "6" smd roundrect
-			(at 1.1375 0.95 90)
+			(at 1.1375 0.95)
 			(size 1.325 0.6)
 			(layers "B.Cu" "B.Mask" "B.Paste")
@@
 	(footprint "All:Pads_1x4"
 		(layer "B.Cu")
-		(at 130.2082 127.9552)
+		(at 142.14 117.87 -90)
 		(property "Reference" "DEBUG_J2"
-			(at -0.3 -1.1 180)
+			(at -0.3 -1.1 90)
 			(unlocked yes)
 			(layer "B.SilkS")
@@
 		)
 		(property "Value" "pads"
-			(at 0 -1 180)
+			(at 0 -1 90)
 			(unlocked yes)
 			(layer "B.Fab")
@@
 		)
 		(property "Datasheet" "~"
-			(at 0 0 180)
+			(at 0 0 90)
 			(unlocked yes)
 			(layer "B.Fab")
@@
 		)
 		(property "Description" "Generic connector, single row, 01x04, script generated"
-			(at 0 0 180)
+			(at 0 0 90)
 			(unlocked yes)
 			(layer "B.Fab")
@@
 		)
 		(fp_line
-			(start 5 -1.25)
-			(end -5 -1.25)
+			(start 5 1.25)
+			(end -5 1.25)
 			(stroke
 				(width 0.05)
@@
 		(fp_line
 			(start 5 1.25)
-			(end -5 1.25)
+			(end 5 -1.25)
 			(stroke
 				(width 0.05)
-				(type default)
+				(type solid)
 			)
 			(layer "B.CrtYd")
 		)
 		(fp_line
-			(start 5 1.25)
-			(end 5 -1.25)
+			(start 5 -1.25)
+			(end -5 -1.25)
 			(stroke
 				(width 0.05)
-				(type solid)
+				(type default)
 			)
 			(layer "B.CrtYd")
 		)
 		(pad "1" smd roundrect
-			(at -3.75 0 180)
+			(at -3.75 0 90)
 			(size 1.6 1.6)
 			(layers "B.Cu" "B.Mask" "B.Paste")
@@
 		)
 		(pad "2" smd roundrect
-			(at -1.25 0 180)
+			(at -1.25 0 90)
 			(size 1.6 1.6)
 			(layers "B.Cu" "B.Mask" "B.Paste")
@@
 		)
 		(pad "3" smd roundrect
-			(at 1.25 0 180)
+			(at 1.25 0 90)
 			(size 1.6 1.6)
 			(layers "B.Cu" "B.Mask" "B.Paste")
@@
 		)
 		(pad "4" smd roundrect
-			(at 3.75 0 180)
+			(at 3.75 0 90)
 			(size 1.6 1.6)
 			(layers "B.Cu" "B.Mask" "B.Paste")

Commit message: layout
Parts:
- removed MCU_C7: 100n, Capacitor_SMD:C_0603_1608Metric_Pad1.08x0.95mm_HandSolder
- removed MCU_C8: 1u, Capacitor_SMD:C_0603_1608Metric_Pad1.08x0.95mm_HandSolder
- 3.3V_R1, 3.3V_R2, 3.3V_R3, 3V3_R0, USB_R0: moved to B.Cu
- ADC_C1, ADC_R1, ADC_R2, DEBUG_J2, FLASH_C1, FLASH_R1, FLASH_R2, U_FLASH1: moved to F.Cu
- J1: value USB4730-GF-A_REVA -> USB4730-GF-A
- moved 3.3V_R1 72.9 mm to (179.3, 130.9), turned to 180 degrees
- moved 3.3V_R2 71.3 mm to (179.3, 129.4), turned to 180 degrees
- moved 3.3V_R3 69.8 mm to (179.3, 128.0), turned to 180 degrees
- moved 3V3_R0 67.0 mm to (179.3, 122.1), turned to 180 degrees
- moved 5V_R0 64.0 mm to (179.3, 125.0), turned to 180 degrees
- moved 3v3_C1 64.0 mm to (176.2, 125.1), turned to 90 degrees
- moved 3V3_C2 60.8 mm to (171.6, 125.1), turned to 90 degrees
- moved 9V_R0 58.9 mm to (179.3, 126.5), turned to 180 degrees
- moved FLASH_C1 54.3 mm to (174.9, 134.4), turned to 180 degrees
- moved FLASH_R1 53.8 mm to (174.9, 135.8), turned to 180 degrees
- moved FLASH_R2 53.4 mm to (174.9, 137.3), turned to 180 degrees
- moved USB_R0 45.5 mm to (179.3, 123.6), turned to 180 degrees
- moved U_FLASH1 43.2 mm to (172.9, 130.4), turned to 0 degrees
- moved ADC_R1 42.0 mm to (155.1, 132.9)
- moved ADC_C1 41.7 mm to (155.1, 130.0), turned to 180 degrees
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Connections:
- net VREF+ renamed 3.3VA
- J1 pad A6: /DP -> unconnected-(J1-DP1-PadA6)
- J1 pad A7: /DN -> unconnected-(J1-DN1-PadA7)
- U2 pad 1: /DP -> /DN
- U2 pad 3: /DN -> /DP
- USB_R3 pad 1: USB_D- -> USB_D+
- USB_R4 pad 1: USB_D+ -> USB_D-
Routing:
- net 3.3V: track 0.00 -> 20.5 mm, vias 0 -> 1
- net 9V_REG: track 0.00 -> 17.2 mm, vias 0 -> 2
- net 5V_REG: track 0.00 -> 17.2 mm, vias 0 -> 2
- net Net-(U_STM32-NRST): track 0.00 -> 11.9 mm
- net Net-(U1-FB): track 0.00 -> 11.3 mm
- net Net-(U3-FB): track 0.00 -> 11.3 mm
- net BAT: track 0.00 -> 9.89 mm, vias 0 -> 1
- net Net-(U3-SW): track 0.00 -> 8.68 mm
- net Net-(U1-SW): track 0.00 -> 8.68 mm
- net Net-(U1-EN): track 0.00 -> 7.94 mm
- net Net-(U3-EN): track 0.00 -> 7.94 mm
- net 3.3VA: track 0.00 -> 7.10 mm
- net BOOT0: track 0.00 -> 5.59 mm
- net Net-(MCU_C14-Pad1): track 0.00 -> 4.13 mm
- net Net-(U1-BOOT): track 0.00 -> 4.02 mm
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- added copper zone on In1.Cu, net GND
- added copper zone on In2.Cu, net GND

Commit message: min
Parts:
- moved 9V_C11 8.21 mm to (133.7, 99.3)
- moved 9V_C12 8.21 mm to (137.0, 109.3)
- moved 9V_C8 8.21 mm to (137.0, 99.3)
- moved 9V_C9 8.21 mm to (137.0, 107.9)
- moved 9V_R5 8.21 mm to (137.0, 100.7)
- moved 9V_R6 8.21 mm to (137.0, 106.4)
- moved 9V_R7 8.21 mm to (137.0, 110.8)
- moved 9V_R8 8.21 mm to (137.0, 112.3)
- moved U3 8.21 mm to (137.0, 103.6)
- moved 9V_C10 8.21 mm to (133.7, 107.9)
- moved 9V_L1 8.21 mm to (130.9, 103.6)
- moved 9V_C7 8.21 mm to (137.0, 97.8)

Commit message: Removed EN resistors from bucks.
Connections:
- U1 pad 5: Net-(U1-EN) -> unconnected-(U1-EN-Pad5)
- U3 pad 5: Net-(U3-EN) -> unconnected-(U3-EN-Pad5)
Changed lines of the file:
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@@
 	(net 127 "unconnected-(J1-DN1-PadA7)")
 	(net 128 "3.3VA")
+	(net 129 "unconnected-(U1-EN-Pad5)")
+	(net 130 "unconnected-(U3-EN-Pad5)")
 	(footprint "Resistor_SMD:R_0603_1608Metric_Pad0.98x0.95mm_HandSolder"
 		(layer "F.Cu")
@@
 			(layers "B.Cu" "B.Mask" "B.Paste")
 			(roundrect_rratio 0.25)
-			(net 20 "Net-(U3-EN)")
+			(net 130 "unconnected-(U3-EN-Pad5)")
 			(pinfunction "EN")
-			(pintype "input")
+			(pintype "input+no_connect")
 		)
 		(pad "6" smd roundrect
@@
 			(layers "B.Cu" "B.Mask" "B.Paste")
 			(roundrect_rratio 0.25)
-			(net 14 "Net-(U1-EN)")
+			(net 129 "unconnected-(U1-EN-Pad5)")
 			(pinfunction "EN")
-			(pintype "input")
+			(pintype "input+no_connect")
 		)
 		(pad "6" smd roundrect
